Commit message: add cylinder

File: urdf/cob4-25_0326.urdf (robot description, URDF)
Before this commit: robot cob4-25, 14 links, 13 joints
Links:
- link fl_caster_r_wheel_link: geometry visual mesh filename=file:///home/nhg-yc/ros2_ws/tricycle_ws/install/tricycle_si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

Commit message: fix mesh

File: urdf/cob4-25_0326.urdf (robot description, URDF)
Before this commit: robot cob4-25, 14 links, 13 joints
Links:
- link fl_caster_r_wheel_link: geometry collision mesh filename=file:///home/nhg-yc/ros2_ws/tricycle_ws/install/tricycle_si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; visual mesh filename=file:///home/nhg-yc/ros2_ws/tricycle_ws/install/tricycle_si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
