Commit message: load world and place tricycle at 10,10,0

File: urdf/min_tricycle_imu_0404.xacro.urdf (robot description, URDF)
Before this commit: robot tricycle_drive, 8 links, 7 joints
Links:
- added link base_footprint
- added link odom
Joints:
- added joint base_joint: type fixed, parent base_link, child base_footprint, origin xyz=0 0 0 rpy=0 0 0
- added joint odom_joint: type fixed, parent base_link, child odom, origin xyz=0.0 0.0 0.0 rpy=0 0 0
