Commit message: fix laser angle in 0408.urdf

File: urdf/cob4-25_0408.urdf (robot description, URDF)
Before this commit: robot tricycle_drive, 13 links, 12 joints
Joints:
- joint base_laser_front_joint: origin xyz=-0.244 0.0 0.20858 rpy=0.0 0.0 0.0 -> xyz=-0.244 0.0 0.20858 rpy=0.0 0.0 3.14
- joint base_laser_left_joint: origin xyz=0.122 0.21131 0.20858 rpy=0.0 0.0 2.094 -> xyz=0.122 0.21131 0.20858 rpy=0.0 0.0 1.0472
- joint base_laser_right_joint: origin xyz=0.122 -0.21131 0.20858 rpy=0.0 0.0 -2.094 -> xyz=0.122 -0.21131 0.20858 rpy=0.0 0.0 -1.0472
