Commit message: add laser for minimum_tri_drive

File: urdf/test_tricycle_drive.xacro.urdf (robot description, URDF)
Before this commit: robot tricycle_drive, 6 links, 5 joints
Links:
- added link base_footprint
- added link imu_link; collision box size=0.1 0.1 0.1; visual box size=0.1 0.1 0.1
- added link lidar_link, mass 0.125; collision cylinder length=0.055 radius=0.0508; visual cylinder length=0.055 radius=0.0508
Joints:
- added joint base_footprint_joint: type fixed, parent base_link, child base_footprint, origin xyz=0 0 0 rpy=0 0 0
- added joint imu_joint: type fixed, parent chassis, child imu_link, origin xyz=0 0 0.01
- added joint lidar_joint: type fixed, parent chassis, child lidar_link, origin xyz=0 0 0.27 rpy=0 0 0
