Commit message: add imu & fix footprint

File: urdf/cob4-25_drive_0409.urdf (robot description, URDF)
Before this commit: robot tricycle_drive, 13 links, 12 joints
Links:
- added link imu_link; collision box size=0.1 0.1 0.1; visual box size=0.1 0.1 0.1
Joints:
- added joint imu_joint: type fixed, parent base_chassis_link, child imu_link, origin xyz=0 0 0.2
- joint base_footprint_joint: child base_link -> base_footprint; parent base_footprint -> base_link
